File: Hardware/TinyFreq.kicad_pcb (KiCad board)
At the start: 2 copper layers, 23.1 x 48.1 mm, 17 parts, among them J1 Edge Connector, J2 ISP, Q1 2N7000, Q2 2N7000, U1 L78L05_TO92, U2 ATtiny85-20S

Commit message: Update schematic datasheets and symbols for TVS diodes, update PCB footprints to reflect the pin change.
Parts:
- moved D3 7.62 mm to (139.9, 109.9), turned to 90 degrees
- moved D2 7.56 mm to (135.4, 109.8), turned to 90 degrees
- moved D4 7.56 mm to (139.7, 95.1), turned to 180 degrees
Connections:
- D2 pad 1: Net-(C1-Pad1) -> Net-(J1-Pad4)
- D2 pad 2: Net-(D2-Pad2) -> Net-(C1-Pad1)
- D3 pad 1: Net-(C1-Pad1) -> Net-(J1-Pad6)
- D3 pad 2: Net-(D3-Pad2) -> Net-(C1-Pad1)
- D4 pad 1: Net-(C1-Pad1) -> Net-(C2-Pad1)
- D4 pad 2: Net-(C2-Pad1) -> Net-(C1-Pad1)
- J1 pad 4: Net-(D2-Pad2) -> Net-(J1-Pad4)
- J1 pad 6: Net-(D3-Pad2) -> Net-(J1-Pad6)
- R2 pad 2: Net-(D3-Pad2) -> Net-(J1-Pad6)
- R6 pad 2: Net-(D2-Pad2) -> Net-(J1-Pad4)
Routing:
- net Net-(J1-Pad6): track 0.00 -> 28.8 mm
- net Net-(D3-Pad2): track 28.8 -> 0.00 mm
- net Net-(J1-Pad4): track 0.00 -> 18.7 mm
- net Net-(D2-Pad2): track 18.7 -> 0.00 mm

Commit message: Generated gerberfiles, updated readme.
Other:
- board text added: "EDGE CONNECTOR"
Changed lines of the file:
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@@
       (outputformat 1)
       (mirror false)
-      (drillshape 1)
+      (drillshape 0)
       (scaleselection 1)
-      (outputdirectory "")
+      (outputdirectory "Gerbers/")
     )
   )
@@
     (effects (font (size 0.5 0.5) (thickness 0.1)))
   )
+  (gr_text "EDGE CONNECTOR\n" (at 135.905 134.08) (layer "F.Fab")
+    (effects (font (size 1.5 1.5) (thickness 0.3)))
+  )
   (segment (start 133.155 116.845) (end 133.5 116.5) (width 0.25) (layer "F.Cu") (net 1))

Commit message: Updated Schematic/PCB Reference values, update readme, zip gerbers.
Parts:
- removed R5, R6: 10k, Resistor_THT:R_Axial_DIN0204_L3.6mm_D1.6mm_P5.08mm_Horizontal
- added R1: 100, Resistor_THT:R_Axial_DIN0204_L3.6mm_D1.6mm_P5.08mm_Horizontal, F.Cu at (127.5, 105.0)
- added R3: 10k, Resistor_THT:R_Axial_DIN0204_L3.6mm_D1.6mm_P5.08mm_Horizontal, F.Cu at (127.9, 86.4)
- R2: value 100 -> 10k
- moved R2 3.91 mm to (131.4, 105.0)
Connections:
- D2 pad 1: Net-(J1-Pad4) -> Net-(D2-Pad1)
- D3 pad 1: Net-(J1-Pad6) -> Net-(D3-Pad1)
- J1 pad 4: Net-(J1-Pad4) -> Net-(D2-Pad1)
- J1 pad 6: Net-(J1-Pad6) -> Net-(D3-Pad1)
- R2 pad 1: Net-(C1-Pad2) -> Net-(Q2-Pad2)
- R2 pad 2: Net-(J1-Pad6) -> Net-(D2-Pad1)
Routing:
- net Net-(J1-Pad6): track 28.8 -> 0.00 mm
- net Net-(D3-Pad1): track 0.00 -> 28.8 mm
- net Net-(J1-Pad4): track 18.7 -> 0.00 mm
- net Net-(D2-Pad1): track 0.00 -> 18.7 mm
