File: Hardware/TinyFreq.kicad_sch (KiCad schematic)
At the start: 17 parts, among them J1 Edge Connector, J2 ISP, Q1 2N7000, Q2 2N7000, U1 L78L05_TO92, U2 ATtiny85-20S

Commit message: Update schematic datasheets and symbols for TVS diodes, update PCB footprints to reflect the pin change.
Parts:
- C1: now left out of the parts list
- D2, D3, D4: symbol Device:D_TVS -> Device:D_Zener
Connections:
- net at C1.1, C2.2, C3.2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: now also D2.2 (A), D3.2 (A), D4.2 (A); no longer D2.1 (A1), D3.1 (A1), D4.1 (A1)
- net at C2.1, D1.1 (K), J1.10 (K)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: now also D4.1 (K); no longer D4.2 (A2)
- net at J1.4 (D), R6.2: now also D2.1 (K); no longer D2.2 (A2)
- net at J1.6 (F), R2.2: now also D3.1 (K); no longer D3.2 (A2)
Other:
- moved on the sheet: D2, D3, D4
Changed lines of the file:
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@@
   (junction (at 121.92 88.9) (diameter 0) (color 0 0 0 0)
   )
+  (junction (at 151.13 110.49) (diameter 0) (color 0 0 0 0)
+  )
+  (junction (at 160.02 93.98) (diameter 0) (color 0 0 0 0)
+  )
+  (junction (at 160.02 110.49) (diameter 0) (color 0 0 0 0)
+  )
+  (junction (at 149.86 82.55) (diameter 0) (color 0 0 0 0)
+  )
+  (junction (at 124.46 91.44) (diameter 0) (color 0 0 0 0)
+  )
+  (junction (at 116.84 82.55) (diameter 0) (color 0 0 0 0)
+  )
+  (junction (at 149.86 74.93) (diameter 0) (color 0 0 0 0)
+  )
+  (junction (at 139.7 82.55) (diameter 0) (color 0 0 0 0)
+  )
+  (junction (at 200.66 86.36) (diameter 0) (color 0 0 0 0)
+  )
+  (junction (at 172.72 110.49) (diameter 0) (color 0 0 0 0)
+  )
+  (junction (at 139.7 110.49) (diameter 0) (color 0 0 0 0)
+  )
+  (junction (at 116.84 74.93) (diameter 0) (color 0 0 0 0)
+  )
+  (junction (at 184.15 110.49) (diameter 0) (color 0 0 0 0)
+  )
   (junction (at 194.31 110.49) (diameter 0) (color 0 0 0 0)
   )
-  (junction (at 151.13 110.49) (diameter 0) (color 0 0 0 0)
-  )
-  (junction (at 160.02 93.98) (diameter 0) (color 0 0 0 0)
-  )
-  (junction (at 160.02 110.49) (diameter 0) (color 0 0 0 0)
-  )
-  (junction (at 172.72 110.49) (diameter 0) (color 0 0 0 0)
-  )
-  (junction (at 184.15 110.49) (diameter 0) (color 0 0 0 0)
-  )
-  (junction (at 149.86 82.55) (diameter 0) (color 0 0 0 0)
-  )
-  (junction (at 124.46 91.44) (diameter 0) (color 0 0 0 0)
-  )
-  (junction (at 116.84 82.55) (diameter 0) (color 0 0 0 0)
-  )
-  (junction (at 149.86 74.93) (diameter 0) (color 0 0 0 0)
-  )
-  (junction (at 139.7 82.55) (diameter 0) (color 0 0 0 0)
-  )
-  (junction (at 200.66 86.36) (diameter 0) (color 0 0 0 0)
-  )
-  (junction (at 139.7 110.49) (diameter 0) (color 0 0 0 0)
-  )
-  (junction (at 116.84 74.93) (diameter 0) (color 0 0 0 0)
+  (wire (pts (xy 194.31 110.49) (xy 203.2 110.49))
+    (stroke (width 0) (type default) (color 0 0 0 0))
   )
   (wire (pts (xy 149.86 76.2) (xy 149.86 74.93))
@@
     (stroke (width 0) (type default) (color 0 0 0 0))
   )
+  (wire (pts (xy 172.72 110.49) (xy 184.15 110.49))
+    (stroke (width 0) (type default) (color 0 0 0 0))
+  )
+  (wire (pts (xy 160.02 109.22) (xy 160.02 110.49))
+    (stroke (width 0) (type default) (color 0 0 0 0))
+  )
+  (wire (pts (xy 139.7 82.55) (xy 149.86 82.55))
+    (stroke (width 0) (type default) (color 0 0 0 0))
+  )
+  (wire (pts (xy 115.57 88.9) (xy 121.92 88.9))
+    (stroke (width 0) (type default) (color 0 0 0 0))
+  )
+  (wire (pts (xy 184.15 76.2) (xy 184.15 86.36))
+    (stroke (width 0) (type default) (color 0 0 0 0))
+  )
+  (wire (pts (xy 116.84 99.06) (xy 116.84 82.55))
+    (stroke (width 0) (type default) (color 0 0 0 0))
+  )
+  (wire (pts (xy 121.92 77.47) (xy 125.73 77.47))
+    (stroke (width 0) (type default) (color 0 0 0 0))
+  )
+  (wire (pts (xy 158.75 101.6) (xy 162.56 101.6))
+    (stroke (width 0) (type default) (color 0 0 0 0))
+  )
+  (wire (pts (xy 121.92 88.9) (xy 143.51 88.9))
+    (stroke (width 0) (type default) (color 0 0 0 0))
+  )
+  (wire (pts (xy 151.13 106.68) (xy 151.13 110.49))
+    (stroke (width 0) (type default) (color 0 0 0 0))
+  )
   (wire (pts (xy 184.15 110.49) (xy 194.31 110.49))
     (stroke (width 0) (type default) (color 0 0 0 0))
   )
-  (wire (pts (xy 160.02 109.22) (xy 160.02 110.49))
-    (stroke (width 0) (type default) (color 0 0 0 0))
-  )
-  (wire (pts (xy 139.7 82.55) (xy 149.86 82.55))
-    (stroke (width 0) (type default) (color 0 0 0 0))
-  )
-  (wire (pts (xy 115.57 88.9) (xy 121.92 88.9))
-    (stroke (width 0) (type default) (color 0 0 0 0))
-  )
-  (wire (pts (xy 184.15 76.2) (xy 184.15 86.36))
-    (stroke (width 0) (type default) (color 0 0 0 0))
-  )
-  (wire (pts (xy 116.84 99.06) (xy 116.84 82.55))
-    (stroke (width 0) (type default) (color 0 0 0 0))
-  )
-  (wire (pts (xy 121.92 77.47) (xy 125.73 77.47))
-    (stroke (width 0) (type default) (color 0 0 0 0))
-  )
-  (wire (pts (xy 158.75 101.6) (xy 162.56 101.6))
-    (stroke (width 0) (type default) (color 0 0 0 0))
-  )
-  (wire (pts (xy 121.92 88.9) (xy 143.51 88.9))
-    (stroke (width 0) (type default) (color 0 0 0 0))
-  )
-  (wire (pts (xy 151.13 106.68) (xy 151.13 110.49))
-    (stroke (width 0) (type default) (color 0 0 0 0))
-  )
-  (wire (pts (xy 194.31 110.49) (xy 203.2 110.49))
-    (stroke (width 0) (type default) (color 0 0 0 0))
-  )
   (wire (pts (xy 151.13 88.9) (xy 152.4 88.9))
     (stroke (width 0) (type default) (color 0 0 0 0))
@@
   )
   (wire (pts (xy 115.57 91.44) (xy 124.46 91.44))
-    (stroke (width 0) (type default) (color 0 0 0 0))
-  )
-  (wire (pts (xy 172.72 110.49) (xy 184.15 110.49))
     (stroke (width 0) (type default) (color 0 0 0 0))
   )
@@
     (pin "2")
   )
-  (symbol (lib_id "Device:D_TVS") (at 184.15 106.68 90) (unit 1)
+  (symbol (lib_id "Device:D_Zener") (at 184.15 106.68 270) (unit 1)
     (in_bom yes) (on_board yes) (fields_autoplaced)
     (property "Reference" "D2" (id 0) (at 186.69 105.4099 90)
-      (effects (font (size 1.27 1.27)) (justify right))
+      (effects (font (size 1.27 1.27)) (justify left))
     )
     (property "Value" "SA16A" (id 1) (at 186.69 107.9499 90)
-      (effects (font (size 1.27 1.27)) (justify right))
+      (effects (font (size 1.27 1.27)) (justify left))
     )
     (property "Footprint" "Diode_THT:D_A-405_P7.62mm_Horizontal" (id 2) (at 184.15 106.68 0)
       (effects (font (size 1.27 1.27)) hide)
     )
-    (property "Datasheet" "~" (id 3) (at 184.15 106.68 0)
+    (property "Datasheet" "https://www.littelfuse.com/assetdocs/tvs-diodes-sa-datasheet?assetguid=93214550-6aff-4192-8ecd-8094a6f7cc98" (id 3) (at 184.15 106.68 0)
       (effects (font (size 1.27 1.27)) hide)
     )
@@
     (pin "2")
   )
-  (symbol (lib_id "Device:D_TVS") (at 172.72 106.68 90) (unit 1)
+  (symbol (lib_id "Device:D_Zener") (at 172.72 106.68 270) (unit 1)
     (in_bom yes) (on_board yes) (fields_autoplaced)
     (property "Reference" "D3" (id 0) (at 175.26 105.4099 90)
-      (effects (font (size 1.27 1.27)) (justify right))
+      (effects (font (size 1.27 1.27)) (justify left))
     )
     (property "Value" "SA30A" (id 1) (at 175.26 107.9499 90)
-      (effects (font (size 1.27 1.27)) (justify right))
+      (effects (font (size 1.27 1.27)) (justify left))
     )
     (property "Footprint" "Diode_THT:D_A-405_P7.62mm_Horizontal" (id 2) (at 172.72 106.68 0)
       (effects (font (size 1.27 1.27)) hide)
     )
-    (property "Datasheet" "~" (id 3) (at 172.72 106.68 0)
+    (property "Datasheet" "https://www.littelfuse.com/assetdocs/tvs-diodes-sa-datasheet?assetguid=93214550-6aff-4192-8ecd-8094a6f7cc98" (id 3) (at 172.72 106.68 0)
       (effects (font (size 1.27 1.27)) hide)
     )
@@
   )
   (symbol (lib_id "Device:C_Small") (at 160.02 106.68 180) (unit 1)
-    (in_bom yes) (on_board yes)
+    (in_bom no) (on_board yes)
     (property "Reference" "C1" (id 0) (at 157.48 105.41 0)
       (effects (font (size 1.27 1.27)) (justify left))
@@
     (pin "2")
   )
-  (symbol (lib_id "Device:D_TVS") (at 194.31 106.68 90) (unit 1)
+  (symbol (lib_id "Device:D_Zener") (at 194.31 106.68 270) (unit 1)
     (in_bom yes) (on_board yes) (fields_autoplaced)
     (property "Reference" "D4" (id 0) (at 196.85 105.4099 90)
-      (effects (font (size 1.27 1.27)) (justify right))
+      (effects (font (size 1.27 1.27)) (justify left))
     )
     (property "Value" "SA30A" (id 1) (at 196.85 107.9499 90)
-      (effects (font (size 1.27 1.27)) (justify right))
+      (effects (font (size 1.27 1.27)) (justify left))
     )
     (property "Footprint" "Diode_THT:D_A-405_P7.62mm_Horizontal" (id 2) (at 194.31 106.68 0)
       (effects (font (size 1.27 1.27)) hide)
     )
-    (property "Datasheet" "~" (id 3) (at 194.31 106.68 0)
-      (effects (font (size 1.27 1.27)) hide)
-    )
+    (property "Datasheet" "https://www.littelfuse.com/assetdocs/tvs-diodes-sa-datasheet?assetguid=93214550-6aff-4192-8ecd-8094a6f7cc98" (id 3) (at 194.31 106.68 0)
+      (effects (font (size 1.27 1.27)) hide)
+    )

Commit message: Generated gerberfiles, updated readme.
Parts:
- J2: now left out of the parts list
Changed lines of the file:
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@@
   )
   (symbol (lib_id "Connector_Generic:Conn_02x03_Odd_Even") (at 130.81 80.01 0) (unit 1)
-    (in_bom yes) (on_board yes)
+    (in_bom no) (on_board yes)
     (property "Reference" "J2" (id 0) (at 132.08 85.09 0))
     (property "Value" "ISP" (id 1) (at 132.08 87.63 0))

Commit message: Updated Schematic/PCB Reference values, update readme, zip gerbers.
Parts:
- renumbered R2 to R1, R6 to R2, R5 to R3
Changed lines of the file:
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@@
   (symbol (lib_id "Device:R_US") (at 166.37 101.6 90) (unit 1)
     (in_bom yes) (on_board yes)
-    (property "Reference" "R6" (id 0) (at 166.37 104.14 90))
+    (property "Reference" "R2" (id 0) (at 166.37 104.14 90))
     (property "Value" "10k" (id 1) (at 166.37 106.68 90))
     (property "Footprint" "Resistor_THT:R_Axial_DIN0204_L3.6mm_D1.6mm_P5.08mm_Horizontal" (id 2) (at 166.624 100.584 90)
@@
   (symbol (lib_id "Device:R_US") (at 147.32 88.9 270) (unit 1)
     (in_bom yes) (on_board yes)
-    (property "Reference" "R5" (id 0) (at 147.32 91.44 90))
+    (property "Reference" "R3" (id 0) (at 147.32 91.44 90))
     (property "Value" "10k" (id 1) (at 147.32 93.98 90))
     (property "Footprint" "Resistor_THT:R_Axial_DIN0204_L3.6mm_D1.6mm_P5.08mm_Horizontal" (id 2) (at 147.066 89.916 90)
@@
   (symbol (lib_id "Device:R_US") (at 166.37 93.98 90) (unit 1)
     (in_bom yes) (on_board yes)
-    (property "Reference" "R2" (id 0) (at 166.37 96.52 90))
+    (property "Reference" "R1" (id 0) (at 166.37 96.52 90))
     (property "Value" "100" (id 1) (at 166.37 99.06 90))
     (property "Footprint" "Resistor_THT:R_Axial_DIN0204_L3.6mm_D1.6mm_P5.08mm_Horizontal" (id 2) (at 166.624 92.964 90)
@@
     )
     (path "/5ad76ee9-d22a-4977-9fe3-f53cc3046e1e"
-      (reference "R2") (unit 1) (value "100") (footprint "Resistor_THT:R_Axial_DIN0204_L3.6mm_D1.6mm_P5.08mm_Horizontal")
+      (reference "R1") (unit 1) (value "100") (footprint "Resistor_THT:R_Axial_DIN0204_L3.6mm_D1.6mm_P5.08mm_Horizontal")
+    )
+    (path "/0990bf38-93cd-4680-b1f3-9aa8f7a7fb7e"
+      (reference "R2") (unit 1) (value "10k") (footprint "Resistor_THT:R_Axial_DIN0204_L3.6mm_D1.6mm_P5.08mm_Horizontal")
+    )
+    (path "/1451c18a-2697-4398-be98-795ddefcac69"
+      (reference "R3") (unit 1) (value "10k") (footprint "Resistor_THT:R_Axial_DIN0204_L3.6mm_D1.6mm_P5.08mm_Horizontal")
     )
     (path "/b0b762ba-571b-460b-b2f4-e951ef430218"
       (reference "R4") (unit 1) (value "10k") (footprint "Resistor_THT:R_Axial_DIN0204_L3.6mm_D1.6mm_P5.08mm_Horizontal")
     )
-    (path "/1451c18a-2697-4398-be98-795ddefcac69"
-      (reference "R5") (unit 1) (value "10k") (footprint "Resistor_THT:R_Axial_DIN0204_L3.6mm_D1.6mm_P5.08mm_Horizontal")
-    )
-    (path "/0990bf38-93cd-4680-b1f3-9aa8f7a7fb7e"
-      (reference "R6") (unit 1) (value "10k") (footprint "Resistor_THT:R_Axial_DIN0204_L3.6mm_D1.6mm_P5.08mm_Horizontal")
-    )
     (path "/00dad84e-2b59-4ab3-a10a-0bf5ebd3823c"
